File: WaterValveController/hardware/WaterValveController.kicad_pcb (KiCad board)
At the start: 2 copper layers, 66 x 76 mm, 51 parts, among them J1 12V DC IN, J2 MAIN SWITCH, J3 VALVE / FLOW, J4 ESP32, J5 BUTTON, J6 LED 25L, J7 LED 50L, J8 LED 100L, Q1 IRF9540N, Q2 2N7000, U1 R-78E5.0-1.0 or L7805, U2 RX480E-4

Commit message: Rev 1.3: 3 A fuse, wider power copper, normally open valve, JLCPCB files
- Fuse F1 is now 3 A. The 12 V and valve tracks are 2.5 mm (about 4.6 A for
  a 10 C rise), GND tracks 1.5 mm, power vias 1.2/0.6 mm. On the mixed board
  the 12 V feed to the valve switch runs beside U1 and C2, not through them.
- Both boards rerouted: 0 DRC errors, 0 warnings, 0 unconnected.
- Firmware defaults to a normally open valve (VALVE_NORMALLY_CLOSED = false).
- New tools/make_jlc.py writes a JLCPCB folder per board: gerber zip
  (Protel names, no X2, drill files and maps), BOM (Comment, Designator,
  Footprint, JLCPCB Part #), CPL (Designator, Mid X, Mid Y, Layer, Rotation)
  and an upload README. The main BOMs gain an LCSC column.
- Silkscreen: fixed positions for the R1 (THT) and C10/R2 (mixed) labels,
  smaller back text clear of J2, stitching vias kept out of lettering.

Co-Authored-By: Claude Opus 5.5 <noreply@anthropic.com>
Claude-Session: https://claude.ai/code/session_01AqRGusXgpSip5brBmMU9hY
Parts:
- F1: value 2A blade (ATO) -> 3A blade (ATO)
Routing:
- net +5V: track 199.0 -> 184.2 mm
- net GND: track 282.9 -> 290.3 mm, vias 111 -> 97
- net /RF4: track 36.2 -> 31.5 mm
- net /TO_ESP: track 48.3 -> 52.1 mm
- net Net-(Q1-G): track 38.0 -> 34.8 mm
- net /RX_D1: track 16.0 -> 13.0 mm
- net /RX_D2: track 18.9 -> 20.4 mm
- net +12V: track 86.6 -> 87.9 mm
- net Net-(Q2-G): track 12.3 -> 11.1 mm
Other:
- board text added: "FUSE 3A"
- board text added: "THROUGH-HOLE rev 1.3"
- board text removed: "FUSE 2A"
- board text removed: "THROUGH-HOLE rev 1.2"
