File: WaterValveController/hardware/WaterValveController.kicad_sch (KiCad schematic)
At the start: 50 parts, among them J1 12V DC IN, J2 VALVE POWER, J3 RELAY MODULE, J4 FLOW SENSOR, J5 ESP32-C3, K1 Relay module, SW1 MODE / CAL, U1 R-78E5.0-1.0 or L7805, U2 RX480E-4

Commit message: Add autorouted through-hole and mixed SMD PCBs (rev 1.2)
Circuit changes requested for the PCB:
- On-board high-side P-MOSFET valve driver (Q1, Q2, R18-R20) with the
  flyback diode D2 on the board; no relay module.
- Standard ATO blade fuse holder (Keystone 3557-2) ahead of a 3-way
  MAIN SWITCH terminal for an illuminated rocker switch.
- 4-way VALVE / FLOW terminal (valve +, GND, 5 V, flow signal).
- JST-XH connectors for the panel button and LEDs, and a 4-pin two-way
  ESP32 link (ESP TX -> D12 through 1k for future control).
- M4 mounting holes.

Boards (2 layers, 1 oz, DRC clean, fully routed with Freerouting):
- Through-hole: 66 x 76 mm, flat resistors under the socketed Nano.
- Mixed SMD + THT: 66 x 69.2 mm.
Both keep 12 V in and the switch on one narrow edge and the valve/flow
terminal on the other, 2 mm tracks for 12 V and the valve, GND poured
on both layers, and an 18 x 19 mm heatsink area above the regulator.

tools/gen_pcb.py places, routes, pours, checks and exports each board
from tools/pcb_layout.py; render_pcb.py draws the board images.

Firmware: the valve output is now active-high for the MOSFET driver
(VALVE_DRIVE_ACTIVE_LOW = false; true for a relay module).

Co-Authored-By: Claude Opus 5.5 <noreply@anthropic.com>
Claude-Session: https://claude.ai/code/session_01AqRGusXgpSip5brBmMU9hY
Parts:
- removed C10: 100uF 16V, Capacitor_THT:CP_Radial_D6.3mm_P2.50mm, symbol Device:C_Polarized
- removed C11: 100nF, Capacitor_THT:C_Disc_D5.0mm_W2.5mm_P5.00mm, symbol Device:C
- removed J2: VALVE POWER, TerminalBlock_Phoenix:TerminalBlock_Phoenix_MKDS-1,5-2-5.08_1x02_P5.08mm_Horizontal, symbol Connector:Screw_Terminal_01x02
- removed J3: RELAY MODULE, Connector_PinHeader_2.54mm:PinHeader_1x03_P2.54mm_Vertical, symbol Connector_Generic:Conn_01x03
- removed J4: FLOW SENSOR, TerminalBlock_Phoenix:TerminalBlock_Phoenix_MKDS-1,5-3-5.08_1x03_P5.08mm_Horizontal, symbol Connector:Screw_Terminal_01x03
- removed J5: ESP32-C3, Connector_PinHeader_2.54mm:PinHeader_1x03_P2.54mm_Vertical, symbol Connector_Generic:Conn_01x03
- removed K1: Relay module, symbol WaterValve:Relay_Module
- added C10: 100nF, Capacitor_THT:C_Disc_D5.0mm_W2.5mm_P5.00mm, symbol Device:C
- added J2: MAIN SWITCH, TerminalBlock_Phoenix:TerminalBlock_Phoenix_MKDS-1,5-3-5.08_1x03_P5.08mm_Horizontal, symbol Connector:Screw_Terminal_01x03
- added J3: VALVE / FLOW, TerminalBlock_Phoenix:TerminalBlock_Phoenix_MKDS-1,5-4-5.08_1x04_P5.08mm_Horizontal, symbol Connector:Screw_Terminal_01x04
- added J4: ESP32, Connector_JST:JST_XH_B4B-XH-A_1x04_P2.50mm_Vertical, symbol Connector_Generic:Conn_01x04
- added J5: BUTTON, Connector_JST:JST_XH_B2B-XH-A_1x02_P2.50mm_Vertical, symbol Connector_Generic:Conn_01x02
- added J6: LED 25L, Connector_JST:JST_XH_B2B-XH-A_1x02_P2.50mm_Vertical, symbol Connector_Generic:Conn_01x02
- added J7: LED 50L, Connector_JST:JST_XH_B2B-XH-A_1x02_P2.50mm_Vertical, symbol Connector_Generic:Conn_01x02
- added J8: LED 100L, Connector_JST:JST_XH_B2B-XH-A_1x02_P2.50mm_Vertical, symbol Connector_Generic:Conn_01x02
- added Q1: IRF9540N, Package_TO_SOT_THT:TO-220-3_Vertical, symbol Transistor_FET:IRF9540N
- added Q2: 2N7000, Package_TO_SOT_THT:TO-92_Inline_Wide, symbol Transistor_FET:2N7000
- added R18, R20: 10k, Resistor_THT:R_Axial_DIN0207_L6.3mm_D2.5mm_P2.54mm_Vertical, symbol Device:R
- added R19: 100, Resistor_THT:R_Axial_DIN0207_L6.3mm_D2.5mm_P2.54mm_Vertical, symbol Device:R
- added R21: 1k, Resistor_THT:R_Axial_DIN0207_L6.3mm_D2.5mm_P7.62mm_Horizontal, symbol Device:R
- added SW2: Rocker switch, 12 V lamp, symbol WaterValve:Rocker_Switch_LED
- A1: footprint Module:Arduino_Nano -> WaterValve:Arduino_Nano_Socketed
- D1: footprint Diode_THT:D_DO-201AD_P15.24mm_Horizontal -> Diode_THT:D_DO-201AD_P5.08mm_Vertical_KathodeUp
- D2: footprint (none) -> Diode_THT:D_DO-201AD_P5.08mm_Vertical_KathodeUp
- D3, D4, D5: footprint LED_THT:LED_D5.0mm -> (none)
- F1: value 2A slow -> 2A blade (ATO); footprint Fuse:Fuseholder_Cylinder-5x20mm_Stelvio-Kontek_PTF78_Horizontal_Open -> WaterValve:Fuseholder_Blade_ATO_Keystone_3557-2
- H1, H2, H3, H4: value M3 -> M4; footprint MountingHole:MountingHole_3.2mm_M3 -> MountingHole:MountingHole_4.3mm_M4
- R1, R17, R2, R3, R4, R5, R6: footprint Resistor_THT:R_Axial_DIN0207_L6.3mm_D2.5mm_P10.16mm_Horizontal -> Resistor_THT:R_Axial_DIN0207_L6.3mm_D2.5mm_P2.54mm_Vertical
- R10, R11, R12, R13, R14, R15, R16, R7, R8, R9: footprint Resistor_THT:R_Axial_DIN0207_L6.3mm_D2.5mm_P10.16mm_Horizontal -> Resistor_THT:R_Axial_DIN0207_L6.3mm_D2.5mm_P7.62mm_Horizontal
- SW1: footprint Button_Switch_THT:SW_PUSH_6mm -> (none)
Connections:
- net +12V: now also J2.2 (Pin_2), Q1.3 (S), R18.1, SW2.2 (LOAD); no longer D1.1 (K), F1.2
- net +5V: now also C10.1, J3.3 (Pin_3), J4.1 (Pin_1)
- net BTN: now also J5.1 (Pin_1)
- net FLOW_IN: now also J3.4 (Pin_4)
- net GND: now also C10.2, J2.3 (Pin_3), J3.2 (Pin_2), J4.2 (Pin_2), J5.2 (Pin_2), J6.2 (Pin_2), J7.2 (Pin_2), J8.2 (Pin_2), Q2.1 (S), R20.2, SW2.3 (LAMP-GND)
- net LED100_A: now reaches D5.2 (A), R6.2
- net LED100_A: now also J8.1 (Pin_1)
- net 12V_IN: now reaches F1.1, J1.1 (Pin_1)
- net SOL_OUT: now reaches D2.1 (K), SV1.1 (+)
- net SOL_OUT: now also J3.1 (Pin_1), Q1.2 (D)
- net LED50_A: now reaches D4.2 (A), R5.2
- net LED50_A: now also J7.1 (Pin_1)
- net LED25_A: now reaches D3.2 (A), R4.2
- net LED25_A: now also J6.1 (Pin_1)
- net ESP_IN: now reaches A1.15 (D12)
- net ESP_IN: now also R21.1
- net ESP_DATA renamed TO_ESP
- net TO_ESP: now also J4.3 (Pin_3)
- net RELAY renamed VALVE
- net VALVE: now also R19.1
- new net: J4.4 (Pin_4), R21.2
- new net: Q2.2 (G), R19.2, R20.1
- new net: Q1.1 (G), Q2.3 (D), R18.2
- new net 12V_FUSED: D1.1 (K), F1.2, J2.1 (Pin_1), SW2.1 (POWER)
- no-connect marks 18 -> 16
Other:
- note added: "1. D2 flyback diode at the valve output; Q1 switches the valve + (high side), valve - goes to GND. 2. 2 mm tracks for the 12 V and valve current; GND poured on both layers. 3. Decoupling: C1 + C2 on 12 V, C3 + C4 at U1, C10 at the Nano, C6 at J3. 4. Flow input: R1 10k pull-up, R2 1k + C5 10nF filter, firmware glitch filter. 5. Button: R3 10k + C7 100nF. Remote: R7-R10 1k series, R13-R16 100k pull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"
- note added: "D11 sends status to the ESP; D12 receives from it (ESP control, for later). Nano is powered through its 5V pin (VIN unused)."
- note added: "D8 HIGH: Q2 pulls the Q1 gate low and the valve gets 12 V. R20 keeps the valve off while the Nano starts. D2 clamps the switch-off spike right at the terminal."
- note added: "ESP32 LINK (JST-XH 4-pin)"
- note added: "F1 + D1: if the supply is connected backwards, D1 conducts and blows F1 (the fuse comes before the main switch, so this works with the switch off too). J2 goes to the illuminated rocker switch; without a switch, link J2 pins 1 and 2. U1: the ESP32-C3 Wi-Fi peaks take the 5 V load to about 0.5 A. Use a pin-compatible switching regulator (R-78E5.0-1.0), or an L7805 on a heatsink."
- note added: "J2 -> SW2: 1 = 12 V in (switch power terminal), 2 = 12 V out (switch load terminal), 3 = lamp GND. J3 -> valve: 1 = valve +, 2 = valve -. Valve flyback diode D2 is on the board."
- note added: "MOUNTING HOLES (M4)"
- note added: "OFF-BOARD PARTS (wired to J2, J3, J5-J8; not placed on the PCB)"
- note added: "PANEL BUTTON AND LIMIT LEDS (JST-XH 2-pin connectors)"
- note added: "POWER IN: BLADE FUSE, MAIN SWITCH, REVERSE-POLARITY CROWBAR, 5 V REGULATOR"
- note added: "R2 + C5 filter fast spikes (time constant 10 us); the firmware also ignores pulses < 2 ms apart."
- note added: "VALVE DRIVER (high-side P-MOSFET) AND VALVE / FLOW SENSOR TERMINAL"
- note removed: "1. D2 flyback diode right at the valve terminals (stripe to +). 2. Valve current has its own pair (J2) back to J1: star ground at J1. 3. Decoupling: C1 + C2 on 12 V, C3 + C4 at U1, C10 at J3, C11 at the Nano, C6 at J4. 4. Flow input: R1 10k pull-up, R2 1k + C5 10nF filter, firmware glitch filter. 5. Button: R3 10k + C7 100nF. Remote: R7-R10 1k series, R13-R16 100k pull-downs, receiver supply filt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"
- note removed: "BUTTON AND LIMIT LEDS"
- note removed: "D12 is reserved for a future ESP -> Nano link. Nano is powered through its 5V pin (VIN unused)."
- note removed: "ESP DATA OUT (9600 baud, 3.3 V level)"
- note removed: "ESP32-C3-Zero: J5 5V -> 5V pin, DATA -> GPIO20 (RX), GND -> GND. Its GPIOs are 3.3 V only, so R11 / R12 drop the Nano's 5 V data to 3.2 V."
- note removed: "F1 + D1: if the supply is connected backwards, D1 conducts and blows F1. U1: the ESP32-C3 Wi-Fi peaks take the 5 V load to about 0.5 A. Use a pin-compatible switching regulator (e.g. R-78E5.0-1.0) or a 5 V buck module wired to IN / GND / OUT. An L7805 needs a heatsink."
- note removed: "J2: run the valve +12 V and return as their own pair, and keep them away from the sensor cable. Place J1 and J2 side by side. C10 sits at J3 to steady 5 V when the relay coil switches."
- note removed: "MOUNTING HOLES (M3)"
- note removed: "OFF-BOARD WIRING (connects to J2-J4; not placed on the PCB)"
- note removed: "POWER: 12 V IN, FUSE, REVERSE-POLARITY CROWBAR, 5 V REGULATOR"
- note removed: "R2 + C5 filter fast spikes (time constant 10 us); the firmware also ignores pulses < 2 ms apart. C6 sits right at J4."
- note removed: "RELAY MODULE AND VALVE POWER"
- note removed: "Valve circuit: relay COM <- J2 pin 1 (+12 V), valve - -> J2 pin 2. D2 sits on the valve terminals."

Commit message: Rev 1.3: 3 A fuse, wider power copper, normally open valve, JLCPCB files
- Fuse F1 is now 3 A. The 12 V and valve tracks are 2.5 mm (about 4.6 A for
  a 10 C rise), GND tracks 1.5 mm, power vias 1.2/0.6 mm. On the mixed board
  the 12 V feed to the valve switch runs beside U1 and C2, not through them.
- Both boards rerouted: 0 DRC errors, 0 warnings, 0 unconnected.
- Firmware defaults to a normally open valve (VALVE_NORMALLY_CLOSED = false).
- New tools/make_jlc.py writes a JLCPCB folder per board: gerber zip
  (Protel names, no X2, drill files and maps), BOM (Comment, Designator,
  Footprint, JLCPCB Part #), CPL (Designator, Mid X, Mid Y, Layer, Rotation)
  and an upload README. The main BOMs gain an LCSC column.
- Silkscreen: fixed positions for the R1 (THT) and C10/R2 (mixed) labels,
  smaller back text clear of J2, stitching vias kept out of lettering.

Co-Authored-By: Claude Opus 5.5 <noreply@anthropic.com>
Claude-Session: https://claude.ai/code/session_01AqRGusXgpSip5brBmMU9hY
Parts:
- F1: value 2A blade (ATO) -> 3A blade (ATO)
Changed lines of the file:
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@@
     (title "Water Valve Controller")
     (date "2026-10-12")
-    (rev "1.2")
+    (rev "1.3")
     (company "Arduino Nano carrier board")
     (comment 1 "YF-G1 flow sensor, MOSFET valve driver, RX480E 433 MHz receiver, ESP link")
@@
       (effects (font (size 1.27 1.27)))
     )
-    (property "Value" "2A blade (ATO)" (at 50.8 54.61 90)
+    (property "Value" "3A blade (ATO)" (at 50.8 54.61 90)
       (effects (font (size 1.27 1.27)))
     )

Commit message: JLCPCB files in the format of JLCPCB's KiCad guide and sample BOM
- CPL columns are now Designator, Mid X, Mid Y, Rotation, Layer, in plain
  millimetres with top/bottom, as the Fabrication Toolkit writes them.
- BOM Footprint column uses short package names (0805, SOT-23, SMC), and the
  BOM is also written as .xlsx laid out like JLCPCB's sample BOM.
- Every part carries an "LCSC Part #" field on its schematic symbol and its
  footprint, so the Fabrication Toolkit can regenerate the files in KiCad
  8-10. Part numbers live in tools/jlc_parts.py.
- Rotation corrections use the usual table of the KiCad JLCPCB plugins
  (only SOT-23 applies to these boards, as before).

Co-Authored-By: Claude Opus 5.5 <noreply@anthropic.com>
Claude-Session: https://claude.ai/code/session_01AqRGusXgpSip5brBmMU9hY
Parts:
- C1: LCSC Part # (none) -> C368591
- C10, C2, C3, C6, C7, C9: LCSC Part # (none) -> C84772
- C4: LCSC Part # (none) -> C911212
- C8: LCSC Part # (none) -> C134586
- D1, D2: LCSC Part # (none) -> C2460
- F1: LCSC Part # (none) -> C352820
- J1: LCSC Part # (none) -> C474940
- J2: LCSC Part # (none) -> C474941
- J3: LCSC Part # (none) -> C2827883
- J4: LCSC Part # (none) -> C144395
- J5, J6, J7, J8: LCSC Part # (none) -> C158012
- Q1: LCSC Part # (none) -> C2575
- Q2: LCSC Part # (none) -> C232838
- R1, R18, R20, R3: LCSC Part # (none) -> C57436
- R10, R2, R21, R7, R8, R9: LCSC Part # (none) -> C57435
- R13, R14, R15, R16: LCSC Part # (none) -> C58597
- R17: LCSC Part # (none) -> C57437
- R19: LCSC Part # (none) -> C57438
- R4, R5, R6: LCSC Part # (none) -> C58608
- U1: LCSC Part # (none) -> C3033024
- U2: LCSC Part # (none) -> C6684533
Changed lines of the file:
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@@
+      (effects (font (size 1.27 1.27)) hide)
+    )
+    (property "LCSC Part #" "C474940" (at 30.48 50.8 0)
       (effects (font (size 1.27 1.27)) hide)
     )
@@
     )
     (property "Datasheet" "~" (at 50.8 50.8 90)
+      (effects (font (size 1.27 1.27)) hide)
+    )
+    (property "LCSC Part #" "C352820" (at 50.8 50.8 90)
       (effects (font (size 1.27 1.27)) hide)
     )
@@
       (effects (font (size 1.27 1.27)) hide)
     )
+    (property "LCSC Part #" "C2460" (at 71.12 57.15 90)
+      (effects (font (size 1.27 1.27)) hide)
+    )
     (pin "1")
     (pin "2")
@@
     )
     (property "Datasheet" "~" (at 86.36 53.34 0)
+      (effects (font (size 1.27 1.27)) hide)
+    )
+    (property "LCSC Part #" "C474941" (at 86.36 53.34 0)
       (effects (font (size 1.27 1.27)) hide)
     )
@@
       (effects (font (size 1.27 1.27)) hide)
     )
+    (property "LCSC Part #" "C3033024" (at 116.84 81.28 0)
+      (effects (font (size 1.27 1.27)) hide)
+    )
     (pin "1")
     (pin "2")
@@
       (effects (font (size 1.27 1.27)) hide)
     )
+    (property "LCSC Part #" "C368591" (at 86.36 87.63 0)
+      (effects (font (size 1.27 1.27)) hide)
+    )
     (pin "1")
     (pin "2")
@@
       (effects (font (size 1.27 1.27)) hide)
     )
+    (property "LCSC Part #" "C84772" (at 101.6 87.63 0)
+      (effects (font (size 1.27 1.27)) hide)
+    )
     (pin "1")
     (pin "2")
@@
       (effects (font (size 1.27 1.27)) hide)
     )
+    (property "LCSC Part #" "C84772" (at 132.08 87.63 0)
+      (effects (font (size 1.27 1.27)) hide)
+    )
     (pin "1")
     (pin "2")
@@
     )
     (property "Datasheet" "~" (at 144.78 87.63 0)
+      (effects (font (size 1.27 1.27)) hide)
+    )
+    (property "LCSC Part #" "C911212" (at 144.78 87.63 0)
       (effects (font (size 1.27 1.27)) hide)
     )
@@
       (effects (font (size 1.27 1.27)) hide)
     )
+    (property "LCSC Part #" "C2575" (at 68.58 134.62 0)
+      (effects (font (size 1.27 1.27)) hide)
+    )
     (pin "1")
     (pin "2")
@@
       (effects (font (size 1.27 1.27)) hide)
     )
+    (property "LCSC Part #" "C57436" (at 58.42 130.81 0)
+      (effects (font (size 1.27 1.27)) hide)
+    )
     (pin "1")
     (pin "2")
@@
       (effects (font (size 1.27 1.27)) hide)
     )
+    (property "LCSC Part #" "C232838" (at 55.88 147.32 0)
+      (effects (font (size 1.27 1.27)) hide)
+    )
     (pin "1")
     (pin "2")
@@
       (effects (font (size 1.27 1.27)) hide)
     )
+    (property "LCSC Part #" "C57438" (at 45.72 147.32 90)
+      (effects (font (size 1.27 1.27)) hide)
+    )
     (pin "1")
     (pin "2")
@@
     )
     (property "Datasheet" "~" (at 49.53 151.13 0)
+      (effects (font (size 1.27 1.27)) hide)
+    )
+    (property "LCSC Part #" "C57436" (at 49.53 151.13 0)
       (effects (font (size 1.27 1.27)) hide)
     )
@@
       (effects (font (size 1.27 1.27)) hide)
     )
+    (property "LCSC Part #" "C2460" (at 78.74 146.05 90)
+      (effects (font (size 1.27 1.27)) hide)
+    )
     (pin "1")
     (pin "2")
@@
       (effects (font (size 1.27 1.27)) hide)
     )
+    (property "LCSC Part #" "C2827883" (at 101.6 144.78 0)
+      (effects (font (size 1.27 1.27)) hide)
+    )
     (pin "1")
     (pin "2")
@@
       (effects (font (size 1.27 1.27)) hide)
     )
+    (property "LCSC Part #" "C84772" (at 116.84 146.05 0)
+      (effects (font (size 1.27 1.27)) hide)
+    )
     (pin "1")
     (pin "2")
@@
       (effects (font (size 1.27 1.27)) hide)
     )
+    (property "LCSC Part #" "C57436" (at 30.48 175.26 0)
+      (effects (font (size 1.27 1.27)) hide)
+    )
     (pin "1")
     (pin "2")
@@
     )
     (property "Datasheet" "~" (at 39.37 180.34 90)
+      (effects (font (size 1.27 1.27)) hide)
+    )
+    (property "LCSC Part #" "C57435" (at 39.37 180.34 90)
       (effects (font (size 1.27 1.27)) hide)
     )
@@
       (effects (font (size 1.27 1.27)) hide)
     )
+    (property "LCSC Part #" "C84772" (at 238.76 101.6 0)
+      (effects (font (size 1.27 1.27)) hide)
+    )
     (pin "1")
     (pin "2")
@@
     )
     (property "Datasheet" "~" (at 398.78 63.5 0)
+      (effects (font (size 1.27 1.27)) hide)
+    )
+    (property "LCSC Part #" "C6684533" (at 398.78 63.5 0)
       (effects (font (size 1.27 1.27)) hide)
     )
@@
       (effects (font (size 1.27 1.27)) hide)
     )
+    (property "LCSC Part #" "C57437" (at 365.76 40.64 90)
+      (effects (font (size 1.27 1.27)) hide)
+    )
     (pin "1")
     (pin "2")
@@
       (effects (font (size 1.27 1.27)) hide)
     )
+    (property "LCSC Part #" "C134586" (at 375.92 46.99 0)
+      (effects (font (size 1.27 1.27)) hide)
+    )
     (pin "1")
     (pin "2")
@@
     )
     (property "Datasheet" "~" (at 386.08 46.99 0)
+      (effects (font (size 1.27 1.27)) hide)
+    )
+    (property "LCSC Part #" "C84772" (at 386.08 46.99 0)
       (effects (font (size 1.27 1.27)) hide)
     )
@@
       (effects (font (size 1.27 1.27)) hide)
     )
+    (property "LCSC Part #" "C57435" (at 289.56 46.99 0)
+      (effects (font (size 1.27 1.27)) hide)
+    )
     (pin "1")
     (pin "2")
@@
     )
     (property "Datasheet" "~" (at 289.56 59.69 0)
+      (effects (font (size 1.27 1.27)) hide)
+    )
+    (property "LCSC Part #" "C58597" (at 289.56 59.69 0)
       (effects (font (size 1.27 1.27)) hide)
     )
@@
       (effects (font (size 1.27 1.27)) hide)
     )
+    (property "LCSC Part #" "C57435" (at 307.34 46.99 0)
+      (effects (font (size 1.27 1.27)) hide)
+    )
     (pin "1")
     (pin "2")
@@
     )
     (property "Datasheet" "~" (at 307.34 59.69 0)
+      (effects (font (size 1.27 1.27)) hide)
+    )
+    (property "LCSC Part #" "C58597" (at 307.34 59.69 0)
       (effects (font (size 1.27 1.27)) hide)
     )
@@
       (effects (font (size 1.27 1.27)) hide)
     )
+    (property "LCSC Part #" "C57435" (at 325.12 46.99 0)
+      (effects (font (size 1.27 1.27)) hide)
+    )
     (pin "1")
     (pin "2")
@@
     )
     (property "Datasheet" "~" (at 325.12 59.69 0)
+      (effects (font (size 1.27 1.27)) hide)
+    )
+    (property "LCSC Part #" "C58597" (at 325.12 59.69 0)
       (effects (font (size 1.27 1.27)) hide)
     )
@@
       (effects (font (size 1.27 1.27)) hide)
     )
+    (property "LCSC Part #" "C57435" (at 342.9 46.99 0)
+      (effects (font (size 1.27 1.27)) hide)
+    )
     (pin "1")
     (pin "2")
@@
     )
     (property "Datasheet" "~" (at 342.9 59.69 0)
+      (effects (font (size 1.27 1.27)) hide)
+    )
+    (property "LCSC Part #" "C58597" (at 342.9 59.69 0)
       (effects (font (size 1.27 1.27)) hide)
     )
@@
       (effects (font (size 1.27 1.27)) hide)
     )
+    (property "LCSC Part #" "C57436" (at 289.56 92.71 0)
+      (effects (font (size 1.27 1.27)) hide)
+    )
     (pin "1")
     (pin "2")
@@
       (effects (font (size 1.27 1.27)) hide)
     )
+    (property "LCSC Part #" "C84772" (at 289.56 100.33 0)
+      (effects (font (size 1.27 1.27)) hide)
+    )
     (pin "1")
     (pin "2")
@@
     )
     (property "Datasheet" "~" (at 314.96 96.52 0)
+      (effects (font (size 1.27 1.27)) hide)
+    )
+    (property "LCSC Part #" "C158012" (at 314.96 96.52 0)
       (effects (font (size 1.27 1.27)) hide)
     )
@@
       (effects (font (size 1.27 1.27)) hide)
     )
+    (property "LCSC Part #" "C58608" (at 289.56 116.84 90)
+      (effects (font (size 1.27 1.27)) hide)
+    )
     (pin "1")
     (pin "2")
@@
     )
     (property "Datasheet" "~" (at 314.96 116.84 0)
+      (effects (font (size 1.27 1.27)) hide)
+    )
+    (property "LCSC Part #" "C158012" (at 314.96 116.84 0)
       (effects (font (size 1.27 1.27)) hide)
     )
@@
       (effects (font (size 1.27 1.27)) hide)
     )
+    (property "LCSC Part #" "C58608" (at 289.56 127 90)
+      (effects (font (size 1.27 1.27)) hide)
+    )
     (pin "1")
     (pin "2")
@@
     )
     (property "Datasheet" "~" (at 314.96 127 0)
+      (effects (font (size 1.27 1.27)) hide)
+    )
+    (property "LCSC Part #" "C158012" (at 314.96 127 0)
       (effects (font (size 1.27 1.27)) hide)
     )
@@
       (effects (font (size 1.27 1.27)) hide)
     )
+    (property "LCSC Part #" "C58608" (at 289.56 137.16 90)
+      (effects (font (size 1.27 1.27)) hide)
+    )
     (pin "1")
     (pin "2")
@@
     )
     (property "Datasheet" "~" (at 314.96 137.16 0)
+      (effects (font (size 1.27 1.27)) hide)
+    )
+    (property "LCSC Part #" "C158012" (at 314.96 137.16 0)
       (effects (font (size 1.27 1.27)) hide)
     )
@@
       (effects (font (size 1.27 1.27)) hide)
     )
+    (property "LCSC Part #" "C144395" (at 340.36 161.29 0)
+      (effects (font (size 1.27 1.27)) hide)
+    )
     (pin "1")
     (pin "2")
@@
       (effects (font (size 1.27 1.27)) hide)
     )
+    (property "LCSC Part #" "C57435" (at 326.39 166.37 90)
+      (effects (font (size 1.27 1.27)) hide)
+    )
