File: WaterValveController/hardware/smd/WaterValveController-SMD.kicad_pcb (KiCad board)
At the start: 2 copper layers, 66 x 69.2 mm, 51 parts, among them J1 12V DC IN, J2 MAIN SWITCH, J3 VALVE / FLOW, J4 ESP32, J5 BUTTON, J6 LED 25L, J7 LED 50L, J8 LED 100L, Q1 IRFR5305, Q2 2N7002, U1 R-78E5.0-1.0 or L7805, U2 RX480E-4

Commit message: Rev 1.3: 3 A fuse, wider power copper, normally open valve, JLCPCB files
- Fuse F1 is now 3 A. The 12 V and valve tracks are 2.5 mm (about 4.6 A for
  a 10 C rise), GND tracks 1.5 mm, power vias 1.2/0.6 mm. On the mixed board
  the 12 V feed to the valve switch runs beside U1 and C2, not through them.
- Both boards rerouted: 0 DRC errors, 0 warnings, 0 unconnected.
- Firmware defaults to a normally open valve (VALVE_NORMALLY_CLOSED = false).
- New tools/make_jlc.py writes a JLCPCB folder per board: gerber zip
  (Protel names, no X2, drill files and maps), BOM (Comment, Designator,
  Footprint, JLCPCB Part #), CPL (Designator, Mid X, Mid Y, Layer, Rotation)
  and an upload README. The main BOMs gain an LCSC column.
- Silkscreen: fixed positions for the R1 (THT) and C10/R2 (mixed) labels,
  smaller back text clear of J2, stitching vias kept out of lettering.

Co-Authored-By: Claude Opus 5.5 <noreply@anthropic.com>
Claude-Session: https://claude.ai/code/session_01AqRGusXgpSip5brBmMU9hY
Parts:
- F1: value 2A blade (ATO) -> 3A blade (ATO)
Routing:
- net /TO_ESP: track 58.0 -> 37.1 mm
- net +5V: track 150.1 -> 162.8 mm, vias 2 -> 3
- net /RX_D2: track 22.2 -> 30.4 mm, vias 0 -> 1
- net Net-(Q1-G): track 6.71 -> 13.5 mm
- net +12V: track 81.8 -> 87.9 mm
- net /FLOW_IN: track 33.6 -> 36.3 mm, vias 2 -> 0
- net Net-(Q2-G): track 11.0 -> 13.5 mm, vias 2 -> 0
- net GND: track 294.4 -> 296.9 mm, vias 96 -> 76
- net /BTN: track 35.4 -> 37.7 mm
- net /RX_D1: track 11.3 -> 13.2 mm, vias 1 -> 0
- net Net-(J4-Pin_4): track 34.7 -> 33.2 mm
- net /LED25_A: track 19.5 -> 20.9 mm
- net /LED100_A: track 13.6 -> 14.3 mm, vias 0 -> 2
- net /LED100: track 17.6 -> 16.9 mm
- net /SOL_OUT: track 28.4 -> 29.0 mm
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Other:
- board text added: "FUSE 3A"
- board text added: "MIXED SMD + THT rev 1.3"
- board text removed: "FUSE 2A"
- board text removed: "MIXED SMD + THT rev 1.2"
