File: WaterValveController/hardware/smd/WaterValveController-SMD.kicad_sch (KiCad schematic)
At the start: 58 parts, among them J1 12V DC IN, J2 MAIN SWITCH, J3 VALVE / FLOW, J4 ESP32, J5 BUTTON, J6 LED 25L, J7 LED 50L, J8 LED 100L, Q1 IRFR5305, Q2 2N7002, SW1 MODE / CAL, SW2 Rocker switch, 12 V lamp, U1 R-78E5.0-1.0 or L7805, U2 RX480E-4

Commit message: Rev 1.3: 3 A fuse, wider power copper, normally open valve, JLCPCB files
- Fuse F1 is now 3 A. The 12 V and valve tracks are 2.5 mm (about 4.6 A for
  a 10 C rise), GND tracks 1.5 mm, power vias 1.2/0.6 mm. On the mixed board
  the 12 V feed to the valve switch runs beside U1 and C2, not through them.
- Both boards rerouted: 0 DRC errors, 0 warnings, 0 unconnected.
- Firmware defaults to a normally open valve (VALVE_NORMALLY_CLOSED = false).
- New tools/make_jlc.py writes a JLCPCB folder per board: gerber zip
  (Protel names, no X2, drill files and maps), BOM (Comment, Designator,
  Footprint, JLCPCB Part #), CPL (Designator, Mid X, Mid Y, Layer, Rotation)
  and an upload README. The main BOMs gain an LCSC column.
- Silkscreen: fixed positions for the R1 (THT) and C10/R2 (mixed) labels,
  smaller back text clear of J2, stitching vias kept out of lettering.

Co-Authored-By: Claude Opus 5.5 <noreply@anthropic.com>
Claude-Session: https://claude.ai/code/session_01AqRGusXgpSip5brBmMU9hY
Parts:
- F1: value 2A blade (ATO) -> 3A blade (ATO)
Changed lines of the file:
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@@
     (title "Water Valve Controller")
     (date "2026-10-12")
-    (rev "1.2")
+    (rev "1.3")
     (company "Arduino Nano carrier board")
     (comment 1 "YF-G1 flow sensor, MOSFET valve driver, RX480E 433 MHz receiver, ESP link")
@@
       (effects (font (size 1.27 1.27)))
     )
-    (property "Value" "2A blade (ATO)" (at 50.8 54.61 90)
+    (property "Value" "3A blade (ATO)" (at 50.8 54.61 90)
       (effects (font (size 1.27 1.27)))
     )

Commit message: JLCPCB files in the format of JLCPCB's KiCad guide and sample BOM
- CPL columns are now Designator, Mid X, Mid Y, Rotation, Layer, in plain
  millimetres with top/bottom, as the Fabrication Toolkit writes them.
- BOM Footprint column uses short package names (0805, SOT-23, SMC), and the
  BOM is also written as .xlsx laid out like JLCPCB's sample BOM.
- Every part carries an "LCSC Part #" field on its schematic symbol and its
  footprint, so the Fabrication Toolkit can regenerate the files in KiCad
  8-10. Part numbers live in tools/jlc_parts.py.
- Rotation corrections use the usual table of the KiCad JLCPCB plugins
  (only SOT-23 applies to these boards, as before).

Co-Authored-By: Claude Opus 5.5 <noreply@anthropic.com>
Claude-Session: https://claude.ai/code/session_01AqRGusXgpSip5brBmMU9hY
Parts:
- C1: LCSC Part # (none) -> C368591
- C10, C2, C3, C6, C7, C9: LCSC Part # (none) -> C49678
- C4: LCSC Part # (none) -> C911212
- C5: LCSC Part # (none) -> C1710
- C8: LCSC Part # (none) -> C134586
- D1, D2: LCSC Part # (none) -> C388240
- F1: LCSC Part # (none) -> C352820
- J1: LCSC Part # (none) -> C474940
- J2: LCSC Part # (none) -> C474941
- J3: LCSC Part # (none) -> C2827883
- J4: LCSC Part # (none) -> C144395
- J5, J6, J7, J8: LCSC Part # (none) -> C158012
- Q1: LCSC Part # (none) -> C2624
- Q2: LCSC Part # (none) -> C8545
- R1, R18, R20, R3: LCSC Part # (none) -> C17414
- R10, R2, R21, R7, R8, R9: LCSC Part # (none) -> C17513
- R11: LCSC Part # (none) -> C17398
- R12: LCSC Part # (none) -> C114531
- R13, R14, R15, R16: LCSC Part # (none) -> C149504
- R17: LCSC Part # (none) -> C17415
- R19: LCSC Part # (none) -> C17408
- R4, R5, R6: LCSC Part # (none) -> C17630
- U1: LCSC Part # (none) -> C3033024
- U2: LCSC Part # (none) -> C6684533
Changed lines of the file:
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@@
+      (effects (font (size 1.27 1.27)) hide)
+    )
+    (property "LCSC Part #" "C474940" (at 30.48 50.8 0)
       (effects (font (size 1.27 1.27)) hide)
     )
@@
     )
     (property "Datasheet" "~" (at 50.8 50.8 90)
+      (effects (font (size 1.27 1.27)) hide)
+    )
+    (property "LCSC Part #" "C352820" (at 50.8 50.8 90)
       (effects (font (size 1.27 1.27)) hide)
     )
@@
       (effects (font (size 1.27 1.27)) hide)
     )
+    (property "LCSC Part #" "C388240" (at 71.12 57.15 90)
+      (effects (font (size 1.27 1.27)) hide)
+    )
     (pin "1")
     (pin "2")
@@
     )
     (property "Datasheet" "~" (at 86.36 53.34 0)
+      (effects (font (size 1.27 1.27)) hide)
+    )
+    (property "LCSC Part #" "C474941" (at 86.36 53.34 0)
       (effects (font (size 1.27 1.27)) hide)
     )
@@
       (effects (font (size 1.27 1.27)) hide)
     )
+    (property "LCSC Part #" "C3033024" (at 116.84 81.28 0)
+      (effects (font (size 1.27 1.27)) hide)
+    )
     (pin "1")
     (pin "2")
@@
       (effects (font (size 1.27 1.27)) hide)
     )
+    (property "LCSC Part #" "C368591" (at 86.36 87.63 0)
+      (effects (font (size 1.27 1.27)) hide)
+    )
     (pin "1")
     (pin "2")
@@
       (effects (font (size 1.27 1.27)) hide)
     )
+    (property "LCSC Part #" "C49678" (at 101.6 87.63 0)
+      (effects (font (size 1.27 1.27)) hide)
+    )
     (pin "1")
     (pin "2")
@@
       (effects (font (size 1.27 1.27)) hide)
     )
+    (property "LCSC Part #" "C49678" (at 132.08 87.63 0)
+      (effects (font (size 1.27 1.27)) hide)
+    )
     (pin "1")
     (pin "2")
@@
     )
     (property "Datasheet" "~" (at 144.78 87.63 0)
+      (effects (font (size 1.27 1.27)) hide)
+    )
+    (property "LCSC Part #" "C911212" (at 144.78 87.63 0)
       (effects (font (size 1.27 1.27)) hide)
     )
@@
       (effects (font (size 1.27 1.27)) hide)
     )
+    (property "LCSC Part #" "C2624" (at 68.58 134.62 0)
+      (effects (font (size 1.27 1.27)) hide)
+    )
     (pin "1")
     (pin "2")
@@
       (effects (font (size 1.27 1.27)) hide)
     )
+    (property "LCSC Part #" "C17414" (at 58.42 130.81 0)
+      (effects (font (size 1.27 1.27)) hide)
+    )
     (pin "1")
     (pin "2")
@@
       (effects (font (size 1.27 1.27)) hide)
     )
+    (property "LCSC Part #" "C8545" (at 55.88 147.32 0)
+      (effects (font (size 1.27 1.27)) hide)
+    )
     (pin "1")
     (pin "2")
@@
       (effects (font (size 1.27 1.27)) hide)
     )
+    (property "LCSC Part #" "C17408" (at 45.72 147.32 90)
+      (effects (font (size 1.27 1.27)) hide)
+    )
     (pin "1")
     (pin "2")
@@
     )
     (property "Datasheet" "~" (at 49.53 151.13 0)
+      (effects (font (size 1.27 1.27)) hide)
+    )
+    (property "LCSC Part #" "C17414" (at 49.53 151.13 0)
       (effects (font (size 1.27 1.27)) hide)
     )
@@
       (effects (font (size 1.27 1.27)) hide)
     )
+    (property "LCSC Part #" "C388240" (at 78.74 146.05 90)
+      (effects (font (size 1.27 1.27)) hide)
+    )
     (pin "1")
     (pin "2")
@@
       (effects (font (size 1.27 1.27)) hide)
     )
+    (property "LCSC Part #" "C2827883" (at 101.6 144.78 0)
+      (effects (font (size 1.27 1.27)) hide)
+    )
     (pin "1")
     (pin "2")
@@
       (effects (font (size 1.27 1.27)) hide)
     )
+    (property "LCSC Part #" "C49678" (at 116.84 146.05 0)
+      (effects (font (size 1.27 1.27)) hide)
+    )
     (pin "1")
     (pin "2")
@@
       (effects (font (size 1.27 1.27)) hide)
     )
+    (property "LCSC Part #" "C17414" (at 30.48 175.26 0)
+      (effects (font (size 1.27 1.27)) hide)
+    )
     (pin "1")
     (pin "2")
@@
       (effects (font (size 1.27 1.27)) hide)
     )
+    (property "LCSC Part #" "C17513" (at 39.37 180.34 90)
+      (effects (font (size 1.27 1.27)) hide)
+    )
     (pin "1")
     (pin "2")
@@
     )
     (property "Datasheet" "~" (at 48.26 184.15 0)
+      (effects (font (size 1.27 1.27)) hide)
+    )
+    (property "LCSC Part #" "C1710" (at 48.26 184.15 0)
       (effects (font (size 1.27 1.27)) hide)
     )
@@
       (effects (font (size 1.27 1.27)) hide)
     )
+    (property "LCSC Part #" "C49678" (at 238.76 101.6 0)
+      (effects (font (size 1.27 1.27)) hide)
+    )
     (pin "1")
     (pin "2")
@@
     )
     (property "Datasheet" "~" (at 398.78 63.5 0)
+      (effects (font (size 1.27 1.27)) hide)
+    )
+    (property "LCSC Part #" "C6684533" (at 398.78 63.5 0)
       (effects (font (size 1.27 1.27)) hide)
     )
@@
       (effects (font (size 1.27 1.27)) hide)
     )
+    (property "LCSC Part #" "C17415" (at 365.76 40.64 90)
+      (effects (font (size 1.27 1.27)) hide)
+    )
     (pin "1")
     (pin "2")
@@
       (effects (font (size 1.27 1.27)) hide)
     )
+    (property "LCSC Part #" "C134586" (at 375.92 46.99 0)
+      (effects (font (size 1.27 1.27)) hide)
+    )
     (pin "1")
     (pin "2")
@@
     )
     (property "Datasheet" "~" (at 386.08 46.99 0)
+      (effects (font (size 1.27 1.27)) hide)
+    )
+    (property "LCSC Part #" "C49678" (at 386.08 46.99 0)
       (effects (font (size 1.27 1.27)) hide)
     )
@@
       (effects (font (size 1.27 1.27)) hide)
     )
+    (property "LCSC Part #" "C17513" (at 289.56 46.99 0)
+      (effects (font (size 1.27 1.27)) hide)
+    )
     (pin "1")
     (pin "2")
@@
     )
     (property "Datasheet" "~" (at 289.56 59.69 0)
+      (effects (font (size 1.27 1.27)) hide)
+    )
+    (property "LCSC Part #" "C149504" (at 289.56 59.69 0)
       (effects (font (size 1.27 1.27)) hide)
     )
@@
       (effects (font (size 1.27 1.27)) hide)
     )
+    (property "LCSC Part #" "C17513" (at 307.34 46.99 0)
+      (effects (font (size 1.27 1.27)) hide)
+    )
     (pin "1")
     (pin "2")
@@
     )
     (property "Datasheet" "~" (at 307.34 59.69 0)
+      (effects (font (size 1.27 1.27)) hide)
+    )
+    (property "LCSC Part #" "C149504" (at 307.34 59.69 0)
       (effects (font (size 1.27 1.27)) hide)
     )
@@
       (effects (font (size 1.27 1.27)) hide)
     )
+    (property "LCSC Part #" "C17513" (at 325.12 46.99 0)
+      (effects (font (size 1.27 1.27)) hide)
+    )
     (pin "1")
     (pin "2")
@@
     )
     (property "Datasheet" "~" (at 325.12 59.69 0)
+      (effects (font (size 1.27 1.27)) hide)
+    )
+    (property "LCSC Part #" "C149504" (at 325.12 59.69 0)
       (effects (font (size 1.27 1.27)) hide)
     )
@@
       (effects (font (size 1.27 1.27)) hide)
     )
+    (property "LCSC Part #" "C17513" (at 342.9 46.99 0)
+      (effects (font (size 1.27 1.27)) hide)
+    )
     (pin "1")
     (pin "2")
@@
     )
     (property "Datasheet" "~" (at 342.9 59.69 0)
+      (effects (font (size 1.27 1.27)) hide)
+    )
+    (property "LCSC Part #" "C149504" (at 342.9 59.69 0)
       (effects (font (size 1.27 1.27)) hide)
     )
@@
       (effects (font (size 1.27 1.27)) hide)
     )
+    (property "LCSC Part #" "C17414" (at 289.56 92.71 0)
+      (effects (font (size 1.27 1.27)) hide)
+    )
     (pin "1")
     (pin "2")
@@
       (effects (font (size 1.27 1.27)) hide)
     )
+    (property "LCSC Part #" "C49678" (at 289.56 100.33 0)
+      (effects (font (size 1.27 1.27)) hide)
+    )
     (pin "1")
     (pin "2")
@@
     )
     (property "Datasheet" "~" (at 314.96 96.52 0)
+      (effects (font (size 1.27 1.27)) hide)
+    )
+    (property "LCSC Part #" "C158012" (at 314.96 96.52 0)
       (effects (font (size 1.27 1.27)) hide)
     )
@@
       (effects (font (size 1.27 1.27)) hide)
     )
+    (property "LCSC Part #" "C17630" (at 289.56 116.84 90)
+      (effects (font (size 1.27 1.27)) hide)
+    )
     (pin "1")
     (pin "2")
@@
     )
     (property "Datasheet" "~" (at 314.96 116.84 0)
+      (effects (font (size 1.27 1.27)) hide)
+    )
+    (property "LCSC Part #" "C158012" (at 314.96 116.84 0)
       (effects (font (size 1.27 1.27)) hide)
     )
@@
       (effects (font (size 1.27 1.27)) hide)
     )
+    (property "LCSC Part #" "C17630" (at 289.56 127 90)
+      (effects (font (size 1.27 1.27)) hide)
+    )
     (pin "1")
     (pin "2")
@@
     )
     (property "Datasheet" "~" (at 314.96 127 0)
+      (effects (font (size 1.27 1.27)) hide)
+    )
+    (property "LCSC Part #" "C158012" (at 314.96 127 0)
       (effects (font (size 1.27 1.27)) hide)
     )
@@
       (effects (font (size 1.27 1.27)) hide)
     )
+    (property "LCSC Part #" "C17630" (at 289.56 137.16 90)
+      (effects (font (size 1.27 1.27)) hide)
+    )
     (pin "1")
     (pin "2")
@@
     )
     (property "Datasheet" "~" (at 314.96 137.16 0)
+      (effects (font (size 1.27 1.27)) hide)
+    )
+    (property "LCSC Part #" "C158012" (at 314.96 137.16 0)
       (effects (font (size 1.27 1.27)) hide)
     )
@@
       (effects (font (size 1.27 1.27)) hide)
     )
+    (property "LCSC Part #" "C17398" (at 299.72 160.02 0)
+      (effects (font (size 1.27 1.27)) hide)
+    )
     (pin "1")
     (pin "2")
@@
       (effects (font (size 1.27 1.27)) hide)
     )
+    (property "LCSC Part #" "C114531" (at 299.72 167.64 0)
+      (effects (font (size 1.27 1.27)) hide)
+    )
     (pin "1")
     (pin "2")
@@
     )
     (property "Datasheet" "~" (at 340.36 161.29 0)
+      (effects (font (size 1.27 1.27)) hide)
+    )
+    (property "LCSC Part #" "C144395" (at 340.36 161.29 0)
       (effects (font (size 1.27 1.27)) hide)
     )
@@
       (effects (font (size 1.27 1.27)) hide)
     )
+    (property "LCSC Part #" "C17513" (at 326.39 166.37 90)
+      (effects (font (size 1.27 1.27)) hide)
+    )
