File: hardware/kicad/modules/buzzer/vibeduino-buzzer.kicad_sch (KiCad schematic)
At the start: 7 parts, among them J1 BUS PWR/I2C, J2 BUS SIGNALS, Q1 MMBT3904

Commit message: Add JLCPCB production panel, LCSC part numbers and STEP models
- panel/: all ten modules on one 149.3 x 74.2 mm JLCPCB panel (KiKit):
  5 mm frame, mouse-bite tabs placed automatically clear of copper,
  fiducials on both sides, JLCPCB tooling holes and a JLCJLCJLCJLC
  marker. Panel DRC: 0 errors, 0 unconnected. Includes Gerbers, a
  JLCPCB BOM and CPL (75 placements) and an ordering guide.
- bom.py: LCSC/JLCPCB part numbers for 33 of the 37 kit lines, checked
  against the LCSC/JLCPCB listings; prefers JLCPCB Basic parts. JLCPCB
  BOM/CPL files now cover through-hole parts too, and the CPL applies
  JLCPCB rotation offsets (SOT-23, electrolytic, WS2812B).
- step3d.py + models3d.py: STEP model of every board, a full-stack
  assembly STEP (Uno stand-in + shield + four modules), simple STEP
  models for the parts KiCad's 3D library lacks (RK09K pot, TS-1187A
  switch, JST SH Qwiic, OLED glass), and textured 3D renders made in
  three.js via headless Chromium.
- READMEs and BOM.md describe the panel, LCSC numbers and 3D outputs.

Co-Authored-By: Claude Opus 5.5 <noreply@anthropic.com>
Claude-Session: https://claude.ai/code/session_01M5xoomoyVCZ2jQiwMkFQkx
Parts:
- D1: LCSC (none) -> C2128; MPN 1N4148WS-7-F -> 1N4148WS; Manufacturer Diodes Inc. -> JSCJ
- J1, J2: LCSC (none) -> C492404; MPN — -> PZ254V-11-05P; Manufacturer any -> XFCN
- Q1: LCSC (none) -> C20526; MPN MMBT3904LT1G -> MMBT3904; Manufacturer onsemi -> JSCJ
- R1: LCSC (none) -> C21190
- R2: LCSC (none) -> C25804
Changed lines of the file:
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@@
       )
     )
-    (property "Manufacturer" "any"
+    (property "Manufacturer" "XFCN"
       (at 33.02 49.53 0)
       (effects
@@
       )
     )
-    (property "MPN" "—"
+    (property "MPN" "PZ254V-11-05P"
+      (at 33.02 49.53 0)
+      (effects
+        (font (size 1.27 1.27))
+        hide
+      )
+    )
+    (property "LCSC" "C492404"
       (at 33.02 49.53 0)
       (effects
@@
       )
     )
-    (property "Manufacturer" "any"
+    (property "Manufacturer" "XFCN"
       (at 66.04 49.53 0)
       (effects
@@
       )
     )
-    (property "MPN" "—"
+    (property "MPN" "PZ254V-11-05P"
+      (at 66.04 49.53 0)
+      (effects
+        (font (size 1.27 1.27))
+        hide
+      )
+    )
+    (property "LCSC" "C492404"
       (at 66.04 49.53 0)
       (effects
@@
       )
     )
-    (property "Manufacturer" "onsemi"
+    (property "Manufacturer" "JSCJ"
       (at 99.06 55.88 0)
       (effects
@@
       )
     )
-    (property "MPN" "MMBT3904LT1G"
+    (property "MPN" "MMBT3904"
+      (at 99.06 55.88 0)
+      (effects
+        (font (size 1.27 1.27))
+        hide
+      )
+    )
+    (property "LCSC" "C20526"
       (at 99.06 55.88 0)
       (effects
@@
       )
     )
-    (property "Description" "Passive magnetic buzzer (transducer) 12×9.5 mm, 5 V, 7.6 mm pitch"
+    (property "Description" "Passive magnetic buzzer (transducer) 12×9.5 mm, 5 V, ≥ 40 Ω, 7.6 mm pitch"
       (at 128.27 45.72 0)
       (effects
@@
       )
     )
-    (property "Manufacturer" "Diodes Inc."
+    (property "Manufacturer" "JSCJ"
       (at 165.1 46.99 0)
       (effects
@@
       )
     )
-    (property "MPN" "1N4148WS-7-F"
+    (property "MPN" "1N4148WS"
+      (at 165.1 46.99 0)
+      (effects
+        (font (size 1.27 1.27))
+        hide
+      )
+    )
+    (property "LCSC" "C2128"
       (at 165.1 46.99 0)
       (effects
@@
       )
     )
+    (property "LCSC" "C21190"
+      (at 184.15 53.34 0)
+      (effects
+        (font (size 1.27 1.27))
+        hide
+      )
+    )
     (pin "1")
     (pin "2")
@@
       (at 195.58 54.61 0)
       (effects
+        (font (size 1.27 1.27))
+        hide
+      )
+    )
+    (property "LCSC" "C25804"
+      (at 195.58 54.61 0)
+      (effects
