File: hardware/kicad/modules/dpad/vibeduino-dpad.kicad_sch (KiCad schematic)
At the start: 13 parts, among them J1 BUS PWR/I2C, J2 BUS SIGNALS, SW1 UP, SW2 RIGHT, SW3 DOWN, SW4 LEFT, SW5 A

Commit message: Add JLCPCB production panel, LCSC part numbers and STEP models
- panel/: all ten modules on one 149.3 x 74.2 mm JLCPCB panel (KiKit):
  5 mm frame, mouse-bite tabs placed automatically clear of copper,
  fiducials on both sides, JLCPCB tooling holes and a JLCJLCJLCJLC
  marker. Panel DRC: 0 errors, 0 unconnected. Includes Gerbers, a
  JLCPCB BOM and CPL (75 placements) and an ordering guide.
- bom.py: LCSC/JLCPCB part numbers for 33 of the 37 kit lines, checked
  against the LCSC/JLCPCB listings; prefers JLCPCB Basic parts. JLCPCB
  BOM/CPL files now cover through-hole parts too, and the CPL applies
  JLCPCB rotation offsets (SOT-23, electrolytic, WS2812B).
- step3d.py + models3d.py: STEP model of every board, a full-stack
  assembly STEP (Uno stand-in + shield + four modules), simple STEP
  models for the parts KiCad's 3D library lacks (RK09K pot, TS-1187A
  switch, JST SH Qwiic, OLED glass), and textured 3D renders made in
  three.js via headless Chromium.
- READMEs and BOM.md describe the panel, LCSC numbers and 3D outputs.

Co-Authored-By: Claude Opus 5.5 <noreply@anthropic.com>
Claude-Session: https://claude.ai/code/session_01M5xoomoyVCZ2jQiwMkFQkx
Parts:
- C1: LCSC (none) -> C14663; MPN CL10B104KB8NNNC -> CC0603KRX7R9BB104; Manufacturer Samsung -> YAGEO
- J1, J2: LCSC (none) -> C492404; MPN — -> PZ254V-11-05P; Manufacturer any -> XFCN
- R1, R4, R5: LCSC (none) -> C25804
- R2: LCSC (none) -> C21190
- R3: LCSC (none) -> C22978
- SW1, SW2, SW3, SW4, SW5: LCSC (none) -> C318884; Manufacturer XKB Connectivity -> XKB Connection
Changed lines of the file:
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@@
       )
     )
-    (property "Manufacturer" "any"
+    (property "Manufacturer" "XFCN"
       (at 33.02 49.53 0)
       (effects
@@
       )
     )
-    (property "MPN" "—"
+    (property "MPN" "PZ254V-11-05P"
+      (at 33.02 49.53 0)
+      (effects
+        (font (size 1.27 1.27))
+        hide
+      )
+    )
+    (property "LCSC" "C492404"
       (at 33.02 49.53 0)
       (effects
@@
       )
     )
-    (property "Manufacturer" "any"
+    (property "Manufacturer" "XFCN"
       (at 66.04 49.53 0)
       (effects
@@
       )
     )
-    (property "MPN" "—"
+    (property "MPN" "PZ254V-11-05P"
+      (at 66.04 49.53 0)
+      (effects
+        (font (size 1.27 1.27))
+        hide
+      )
+    )
+    (property "LCSC" "C492404"
       (at 66.04 49.53 0)
       (effects
@@
       )
     )
-    (property "Manufacturer" "XKB Connectivity"
+    (property "Manufacturer" "XKB Connection"
       (at 96.52 48.26 0)
       (effects
@@
     )
     (property "MPN" "TS-1187A-B-A-B"
+      (at 96.52 48.26 0)
+      (effects
+        (font (size 1.27 1.27))
+        hide
+      )
+    )
+    (property "LCSC" "C318884"
       (at 96.52 48.26 0)
       (effects
@@
       )
     )
-    (property "Manufacturer" "XKB Connectivity"
+    (property "Manufacturer" "XKB Connection"
       (at 128.27 48.26 0)
       (effects
@@
     )
     (property "MPN" "TS-1187A-B-A-B"
+      (at 128.27 48.26 0)
+      (effects
+        (font (size 1.27 1.27))
+        hide
+      )
+    )
+    (property "LCSC" "C318884"
       (at 128.27 48.26 0)
       (effects
@@
       )
     )
-    (property "Manufacturer" "XKB Connectivity"
+    (property "Manufacturer" "XKB Connection"
       (at 160.02 48.26 0)
       (effects
@@
     )
     (property "MPN" "TS-1187A-B-A-B"
+      (at 160.02 48.26 0)
+      (effects
+        (font (size 1.27 1.27))
+        hide
+      )
+    )
+    (property "LCSC" "C318884"
       (at 160.02 48.26 0)
       (effects
@@
       )
     )
-    (property "Manufacturer" "XKB Connectivity"
+    (property "Manufacturer" "XKB Connection"
       (at 190.5 48.26 0)
       (effects
@@
     )
     (property "MPN" "TS-1187A-B-A-B"
+      (at 190.5 48.26 0)
+      (effects
+        (font (size 1.27 1.27))
+        hide
+      )
+    )
+    (property "LCSC" "C318884"
       (at 190.5 48.26 0)
       (effects
@@
       )
     )
-    (property "Manufacturer" "XKB Connectivity"
+    (property "Manufacturer" "XKB Connection"
       (at 220.98 48.26 0)
       (effects
@@
     )
     (property "MPN" "TS-1187A-B-A-B"
+      (at 220.98 48.26 0)
+      (effects
+        (font (size 1.27 1.27))
+        hide
+      )
+    )
+    (property "LCSC" "C318884"
       (at 220.98 48.26 0)
       (effects
@@
       )
     )
+    (property "LCSC" "C25804"
+      (at 240.03 53.34 0)
+      (effects
+        (font (size 1.27 1.27))
+        hide
+      )
+    )
     (pin "1")
     (pin "2")
@@
       )
     )
+    (property "LCSC" "C21190"
+      (at 252.73 53.34 0)
+      (effects
+        (font (size 1.27 1.27))
+        hide
+      )
+    )
     (pin "1")
     (pin "2")
@@
       )
     )
+    (property "LCSC" "C22978"
+      (at 264.16 53.34 0)
+      (effects
+        (font (size 1.27 1.27))
+        hide
+      )
+    )
     (pin "1")
     (pin "2")
@@
       )
     )
+    (property "LCSC" "C25804"
+      (at 21.59 82.55 0)
+      (effects
+        (font (size 1.27 1.27))
+        hide
+      )
+    )
     (pin "1")
     (pin "2")
@@
       )
     )
+    (property "LCSC" "C25804"
+      (at 34.29 83.82 0)
+      (effects
+        (font (size 1.27 1.27))
+        hide
+      )
+    )
     (pin "1")
     (pin "2")
@@
       )
     )
-    (property "Manufacturer" "Samsung"
+    (property "Manufacturer" "YAGEO"
       (at 46.99 82.55 0)
       (effects
@@
       )
     )
-    (property "MPN" "CL10B104KB8NNNC"
+    (property "MPN" "CC0603KRX7R9BB104"
       (at 46.99 82.55 0)
       (effects
+        (font (size 1.27 1.27))
+        hide
+      )
+    )
+    (property "LCSC" "C14663"
+      (at 46.99 82.55 0)
+      (effects
