File: hardware/kicad/modules/light/vibeduino-light.kicad_sch (KiCad schematic)
At the start: 5 parts, among them J1 BUS PWR/I2C, J2 BUS SIGNALS

Commit message: Add JLCPCB production panel, LCSC part numbers and STEP models
- panel/: all ten modules on one 149.3 x 74.2 mm JLCPCB panel (KiKit):
  5 mm frame, mouse-bite tabs placed automatically clear of copper,
  fiducials on both sides, JLCPCB tooling holes and a JLCJLCJLCJLC
  marker. Panel DRC: 0 errors, 0 unconnected. Includes Gerbers, a
  JLCPCB BOM and CPL (75 placements) and an ordering guide.
- bom.py: LCSC/JLCPCB part numbers for 33 of the 37 kit lines, checked
  against the LCSC/JLCPCB listings; prefers JLCPCB Basic parts. JLCPCB
  BOM/CPL files now cover through-hole parts too, and the CPL applies
  JLCPCB rotation offsets (SOT-23, electrolytic, WS2812B).
- step3d.py + models3d.py: STEP model of every board, a full-stack
  assembly STEP (Uno stand-in + shield + four modules), simple STEP
  models for the parts KiCad's 3D library lacks (RK09K pot, TS-1187A
  switch, JST SH Qwiic, OLED glass), and textured 3D renders made in
  three.js via headless Chromium.
- READMEs and BOM.md describe the panel, LCSC numbers and 3D outputs.

Co-Authored-By: Claude Opus 5.5 <noreply@anthropic.com>
Claude-Session: https://claude.ai/code/session_01M5xoomoyVCZ2jQiwMkFQkx
Parts:
- C1: LCSC (none) -> C14663; MPN CL10B104KB8NNNC -> CC0603KRX7R9BB104; Manufacturer Samsung -> YAGEO
- J1, J2: LCSC (none) -> C492404; MPN — -> PZ254V-11-05P; Manufacturer any -> XFCN
- R1: LCSC (none) -> C125627; Manufacturer any -> Senba
- R2: LCSC (none) -> C25804
Changed lines of the file:
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@@
       )
     )
-    (property "Manufacturer" "any"
+    (property "Manufacturer" "XFCN"
       (at 33.02 49.53 0)
       (effects
@@
       )
     )
-    (property "MPN" "—"
+    (property "MPN" "PZ254V-11-05P"
+      (at 33.02 49.53 0)
+      (effects
+        (font (size 1.27 1.27))
+        hide
+      )
+    )
+    (property "LCSC" "C492404"
       (at 33.02 49.53 0)
       (effects
@@
       )
     )
-    (property "Manufacturer" "any"
-      (at 66.04 49.53 0)
-      (effects
-        (font (size 1.27 1.27))
-        hide
-      )
-    )
-    (property "MPN" "—"
+    (property "Manufacturer" "XFCN"
+      (at 66.04 49.53 0)
+      (effects
+        (font (size 1.27 1.27))
+        hide
+      )
+    )
+    (property "MPN" "PZ254V-11-05P"
+      (at 66.04 49.53 0)
+      (effects
+        (font (size 1.27 1.27))
+        hide
+      )
+    )
+    (property "LCSC" "C492404"
       (at 66.04 49.53 0)
       (effects
@@
       )
     )
-    (property "Description" "Photoresistor (LDR) 5 mm, 10–20 kΩ @ 10 lux"
-      (at 90.17 53.34 0)
-      (effects
-        (font (size 1.27 1.27))
-        hide
-      )
-    )
-    (property "Manufacturer" "any"
+    (property "Description" "Photoresistor (LDR) 5 mm, 8–20 kΩ @ 10 lux"
+      (at 90.17 53.34 0)
+      (effects
+        (font (size 1.27 1.27))
+        hide
+      )
+    )
+    (property "Manufacturer" "Senba"
       (at 90.17 53.34 0)
       (effects
@@
     )
     (property "MPN" "GL5528"
+      (at 90.17 53.34 0)
+      (effects
+        (font (size 1.27 1.27))
+        hide
+      )
+    )
+    (property "LCSC" "C125627"
       (at 90.17 53.34 0)
       (effects
@@
       )
     )
+    (property "LCSC" "C25804"
+      (at 110.49 53.34 0)
+      (effects
+        (font (size 1.27 1.27))
+        hide
+      )
+    )
     (pin "1")
     (pin "2")
@@
       )
     )
-    (property "Manufacturer" "Samsung"
-      (at 123.19 53.34 0)
-      (effects
-        (font (size 1.27 1.27))
-        hide
-      )
-    )
-    (property "MPN" "CL10B104KB8NNNC"
-      (at 123.19 53.34 0)
-      (effects
+    (property "Manufacturer" "YAGEO"
+      (at 123.19 53.34 0)
+      (effects
+        (font (size 1.27 1.27))
+        hide
+      )
+    )
+    (property "MPN" "CC0603KRX7R9BB104"
+      (at 123.19 53.34 0)
+      (effects
+        (font (size 1.27 1.27))
+        hide
+      )
+    )
+    (property "LCSC" "C14663"
+      (at 123.19 53.34 0)
+      (effects
