File: hardware/kicad/shield/vibeduino-shield.kicad_sch (KiCad schematic)
At the start: 25 parts, among them J1 Arduino POWER, J101 SLOT1 PWR/I2C, J102 SLOT1 SIGNALS, J2 Arduino ANALOG, J201 SLOT2 PWR/I2C, J202 SLOT2 SIGNALS, J3 Arduino DIGITAL_HI, J301 SLOT3 PWR/I2C, J302 SLOT3 SIGNALS, J4 Arduino DIGITAL_LO, J401 SLOT4 PWR/I2C, J402 SLOT4 SIGNALS, J5 QWIIC, Q1 BSS138, Q2 BSS138, SW1 RESET

Commit message: Add JLCPCB production panel, LCSC part numbers and STEP models
- panel/: all ten modules on one 149.3 x 74.2 mm JLCPCB panel (KiKit):
  5 mm frame, mouse-bite tabs placed automatically clear of copper,
  fiducials on both sides, JLCPCB tooling holes and a JLCJLCJLCJLC
  marker. Panel DRC: 0 errors, 0 unconnected. Includes Gerbers, a
  JLCPCB BOM and CPL (75 placements) and an ordering guide.
- bom.py: LCSC/JLCPCB part numbers for 33 of the 37 kit lines, checked
  against the LCSC/JLCPCB listings; prefers JLCPCB Basic parts. JLCPCB
  BOM/CPL files now cover through-hole parts too, and the CPL applies
  JLCPCB rotation offsets (SOT-23, electrolytic, WS2812B).
- step3d.py + models3d.py: STEP model of every board, a full-stack
  assembly STEP (Uno stand-in + shield + four modules), simple STEP
  models for the parts KiCad's 3D library lacks (RK09K pot, TS-1187A
  switch, JST SH Qwiic, OLED glass), and textured 3D renders made in
  three.js via headless Chromium.
- READMEs and BOM.md describe the panel, LCSC numbers and 3D outputs.

Co-Authored-By: Claude Opus 5.5 <noreply@anthropic.com>
Claude-Session: https://claude.ai/code/session_01M5xoomoyVCZ2jQiwMkFQkx
Parts:
- C1: LCSC (none) -> C72475; MPN — -> RVT1C101M0605; Manufacturer any -> ROQANG
- C2, C3: LCSC (none) -> C14663; MPN CL10B104KB8NNNC -> CC0603KRX7R9BB104; Manufacturer Samsung -> YAGEO
- D1: LCSC (none) -> C12624; MPN — -> KT-0603G; Manufacturer any -> Hubei KENTO
- J1, J4: LCSC (none) -> C492407; MPN — -> PZ254V-11-08P; Manufacturer any -> XFCN
- J101, J102, J201, J202, J301, J302, J401, J402: LCSC (none) -> C50950; MPN — -> 2.54-1*5PFemale; Manufacturer any -> BOOMELE
- J2: LCSC (none) -> C492405; MPN — -> PZ254V-11-06P; Manufacturer any -> XFCN
- J3: LCSC (none) -> C492409; MPN — -> PZ254V-11-10P; Manufacturer any -> XFCN
- J5: LCSC (none) -> C160390
- Q1, Q2: LCSC (none) -> C78284; Manufacturer onsemi -> JSCJ
- R1, R2: LCSC (none) -> C23162
- R3, R4: LCSC (none) -> C25804
- R5: LCSC (none) -> C21190
- SW1: LCSC (none) -> C318884; Manufacturer XKB Connectivity -> XKB Connection
