File: usb-led-bar/jst/usb-led-bar-jst.kicad_sch (KiCad schematic)
At the start: 15 parts, among them J1 USB 5V in

Commit message: USB LED bar v2: 8 LEDs, school logo, JST PH and USB-C variants
- Two KiCad projects sharing one footprint library:
  jst/   right-angle JST PH 2.0 socket (S2B-PH-SM4-TB, LCSC C295747)
  usb-c/ HRO TYPE-C-31-M-12 receptacle (LCSC C165948) with separate
         5.1k pull-downs on CC1 and CC2 (LCSC C27834) so USB-C chargers
         and C-to-C cables supply 5 V
- 8 warm-white 2835 LEDs (was 6), 8.65 mm pitch, ~170 mA total
- Banyule Nillumbik Tech School logo as front silkscreen at the right
  end (board-only footprint, strokes >= 0.18 mm); mounting holes removed
  to make room
- Stock 0805 / JST / USB-C footprints copied with 0.16 mm silkscreen
- Both boards DRC clean and match their schematics; per-variant Gerber
  zip, BOM and CPL for JLCPCB; export script handles both variants
- README: ordering steps, USB-A cable + switch suggestions for the JST
  variant, USB-C CC explanation

Co-Authored-By: Claude Opus 5.5 <noreply@anthropic.com>
Claude-Session: https://claude.ai/code/session_013C9F11DiXqXJzCTtebCnow
Parts:
- removed H1, H2: M3, MountingHole:MountingHole_3.2mm_M3, symbol Mechanical:MountingHole
- added D7, D8: Warm White, usb-led-bar:LED_2835_PolarityTolerant, symbol Device:LED
- added R7, R8: 100, usb-led-bar:R_0805_2012Metric, symbol Device:R
- J1: value USB 5V in -> JST PH 2-pin; footprint usb-led-bar:USB_Power_Wires_1x02_P6mm_Relief -> usb-led-bar:JST_PH_S2B-PH-SM4-TB_1x02-1MP_P2.00mm_Horizontal; LCSC (none) -> C295747; MPN (none) -> S2B-PH-SM4-TB(LF)(SN); Manufacturer (none) -> JST; now in the parts list
Connections:
- net +5V: now also R7.1, R8.1
- net GND: now also D7.1 (K), D8.1 (K)
- new net: D7.2 (A), R7.2
- new net: D8.2 (A), R8.2
Other:
- note added: "8 LEDs, each with its own resistor (parallel branches). I(LED) ≈ (5.0 V - 2.9 V) / 100 Ω ≈ 21 mA (typical LED-strip drive current) Total ≈ 168 mA from USB. P(R) ≈ 44 mW (0805 rating 125 mW). D1-D8: XINGLIGHT XL-2835WWC-02 warm white 2835 (2800-3000 K), LCSC C2843875 R1-R8: UNI-ROYAL 0805W8F1000T5E 100R 1% 0805, LCSC C17408"
- note added: "J1: JST PH 2.0 mm right-angle socket (S2B-PH-SM4-TB). Pin 1 = +5V, pin 2 = GND - check the cable before plugging in."
- note removed: "Each LED has its own resistor (6 parallel branches). I(LED) ≈ (5.0 V - 2.9 V) / 100 Ω ≈ 20 mA (typical LED-strip drive current) Total ≈ 125 mA from USB. P(R) ≈ 44 mW (0805 rating 125 mW). D1-D6: XINGLIGHT XL-2835WWC-02 warm white 2835 (2800-3000 K), LCSC C2843875 R1-R6: UNI-ROYAL 0805W8F1000T5E 100R 1% 0805, LCSC C17408"
- note removed: "Mounting holes (M3, no connection)"
- note removed: "USB cable wires: red -> +5V (J1 pin 1) black -> GND (J1 pin 2) (data wires unused - cut them back)"
- company: (none) -> Banyule Nillumbik Tech School

Commit message: Blank underside and M3 mounting hole at the logo end (both variants)
- Remove all back-side silkscreen (title, specs, JLC order-number marker);
  README now says to pick "Remove Mark" when ordering
- Add an M3 hole (3.2 mm NPTH, 6.9 mm head/washer keep-out) between D8
  and the logo; LED pitch 8.65 -> 7.65 mm to make room
- Regenerated schematics, boards (DRC clean, nets match), JLCPCB
  Gerber/BOM/CPL, previews and the USB-C STEP model; make_3d.py skips
  mounting-hole footprints

Co-Authored-By: Claude Opus 5.5 <noreply@anthropic.com>
Claude-Session: https://claude.ai/code/session_013C9F11DiXqXJzCTtebCnow
Parts:
- added H1: M3, MountingHole:MountingHole_3.2mm_M3, symbol Mechanical:MountingHole
Other:
- note added: "M3 mounting hole (logo end, no connection)"
Changed lines of the file:
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@@
+    (effects (font (size 1.27 1.27)) (justify left bottom))
+  )
+  (text "M3 mounting hole\n(logo end, no connection)" (at 241.3 83.82 0)
     (effects (font (size 1.27 1.27)) (justify left bottom))
   )
@@
         )
       )
+    )
+  )
+  (symbol (lib_id "Mechanical:MountingHole") (at 248.92 76.2 0) (unit 1)
+    (in_bom no) (on_board yes) (dnp no)
+    (property "Reference" "H1" (at 248.92 71.12 0)
+      (effects (font (size 1.27 1.27)))
+    )
+    (property "Value" "M3" (at 248.92 73.025 0)
+      (effects (font (size 1.27 1.27)))
+    )
+    (property "Footprint" "MountingHole:MountingHole_3.2mm_M3" (at 248.92 76.2 0)
+      (effects (font (size 1.27 1.27)) hide)
+    )
+    (property "Datasheet" "~" (at 248.92 76.2 0)
+      (effects (font (size 1.27 1.27)) hide)
+    )
+    (instances
+      (project "usb-led-bar-jst"
+        (path "/904bdd59-6204-51e4-883d-f75ec5c3b0c2"
+          (reference "H1") (unit 1)
+        )
+      )
