File: usb-led-bar/usb-c/usb-led-bar-usbc.kicad_pcb (KiCad board)
At the start: 2 copper layers, 100 x 15 mm, 20 parts, among them J1 USB-C (power only)

Commit message: Blank underside and M3 mounting hole at the logo end (both variants)
- Remove all back-side silkscreen (title, specs, JLC order-number marker);
  README now says to pick "Remove Mark" when ordering
- Add an M3 hole (3.2 mm NPTH, 6.9 mm head/washer keep-out) between D8
  and the logo; LED pitch 8.65 -> 7.65 mm to make room
- Regenerated schematics, boards (DRC clean, nets match), JLCPCB
  Gerber/BOM/CPL, previews and the USB-C STEP model; make_3d.py skips
  mounting-hole footprints

Co-Authored-By: Claude Opus 5.5 <noreply@anthropic.com>
Claude-Session: https://claude.ai/code/session_013C9F11DiXqXJzCTtebCnow
Parts:
- added H1: M3, MountingHole:MountingHole_3.2mm_M3, F.Cu at (175.7, 107.5)
- moved D8 7.00 mm to (170.2, 107.5)
- moved R8 7.00 mm to (170.2, 103.2)
- moved D7 6.00 mm to (162.5, 107.5)
- moved R7 6.00 mm to (162.5, 103.2)
- moved D6 5.00 mm to (154.8, 107.5)
- moved R6 5.00 mm to (154.8, 103.2)
- moved D5 4.00 mm to (147.2, 107.5)
- moved R5 4.00 mm to (147.2, 103.2)
- moved D4 3.00 mm to (139.6, 107.5)
- moved R4 3.00 mm to (139.6, 103.2)
- moved D3 2.00 mm to (131.9, 107.5)
- moved R3 2.00 mm to (131.9, 103.2)
- moved D2 1.00 mm to (124.2, 107.5)
- moved R2 1.00 mm to (124.2, 103.2)
Routing:
- net GND: track 110.7 -> 103.7 mm
- net +5V: track 85.2 -> 78.2 mm
Other:
- board text removed: "8x WARM WHITE 2835 LED - 5V ~168mA"
- board text removed: "J1: USB-C 5V input (5.1k CC pull-downs, R9/R10)"
- board text removed: "JLCJLCJLCJLC"
- board text removed: "USB LED BAR v2.0"
