File: usb-led-bar/usb-c/usb-led-bar-usbc.kicad_sch (KiCad schematic)
At the start: 19 parts, among them J1 USB-C (power only)

Commit message: Blank underside and M3 mounting hole at the logo end (both variants)
- Remove all back-side silkscreen (title, specs, JLC order-number marker);
  README now says to pick "Remove Mark" when ordering
- Add an M3 hole (3.2 mm NPTH, 6.9 mm head/washer keep-out) between D8
  and the logo; LED pitch 8.65 -> 7.65 mm to make room
- Regenerated schematics, boards (DRC clean, nets match), JLCPCB
  Gerber/BOM/CPL, previews and the USB-C STEP model; make_3d.py skips
  mounting-hole footprints

Co-Authored-By: Claude Opus 5.5 <noreply@anthropic.com>
Claude-Session: https://claude.ai/code/session_013C9F11DiXqXJzCTtebCnow
Parts:
- added H1: M3, MountingHole:MountingHole_3.2mm_M3, symbol Mechanical:MountingHole
Other:
- note added: "M3 mounting hole (logo end, no connection)"
Changed lines of the file:
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@@
+    (effects (font (size 1.27 1.27)) (justify left bottom))
+  )
+  (text "M3 mounting hole\n(logo end, no connection)" (at 241.3 83.82 0)
     (effects (font (size 1.27 1.27)) (justify left bottom))
   )
@@
         )
       )
+    )
+  )
+  (symbol (lib_id "Mechanical:MountingHole") (at 248.92 76.2 0) (unit 1)
+    (in_bom no) (on_board yes) (dnp no)
+    (property "Reference" "H1" (at 248.92 71.12 0)
+      (effects (font (size 1.27 1.27)))
+    )
+    (property "Value" "M3" (at 248.92 73.025 0)
+      (effects (font (size 1.27 1.27)))
+    )
+    (property "Footprint" "MountingHole:MountingHole_3.2mm_M3" (at 248.92 76.2 0)
+      (effects (font (size 1.27 1.27)) hide)
+    )
+    (property "Datasheet" "~" (at 248.92 76.2 0)
+      (effects (font (size 1.27 1.27)) hide)
+    )
+    (instances
+      (project "usb-led-bar-usbc"
+        (path "/80a6da2f-dfe2-526e-9052-1eecf8e31b4a"
+          (reference "H1") (unit 1)
+        )
+      )
