File: hardware/circuitpath-keychain/kicad/circuitpath-keychain.kicad_sch (KiCad schematic)
At the start: 115 parts, among them J1 USB-A plug (PCB fingers), J2 USB-C (vertical), J3 ISP pads, SW1 Button, SW2 Button, U1 ATmega32U4-AU, U2 MAX7219CWG+T, U3 MAX7219CWG+T, U4 USBLC6-2SC6, Y1 16MHz

Commit message: Keychain: clear logo/text zone before keyring hole, add piezo buzzer, compact layout
Co-Authored-By: Claude Sonnet 5.5 <noreply@anthropic.com>
Claude-Session: https://claude.ai/code/session_01DPLfCi4mjQi9VLJYecUoR3
Parts:
- added BZ1: Piezo 9x9, Buzzer_Beeper:Buzzer_Murata_PKMCS0909E, symbol Device:Buzzer
Connections:
- net BUZZ_A: now reaches U1.29 (PB5)
- net BUZZ_A: now also BZ1.1 (+)
- net BUZZ_B: now reaches U1.30 (PB6)
- net BUZZ_B: now also BZ1.2 (-)
- no-connect marks 26 -> 24

Commit message: Keychain: route board with Freerouting, export Gerbers + drill, DRC-clean at JLCPCB-style limits
Layout fixes found by KiCad DRC: ISP pads without alignment holes, diodes off the corner,
LED row pitch 2.4 mm, CC resistors on back, hand-tied USB-C data pins, edge keep-out band.

Co-Authored-By: Claude Sonnet 5.5 <noreply@anthropic.com>
Claude-Session: https://claude.ai/code/session_01DPLfCi4mjQi9VLJYecUoR3
Parts:
- J3: footprint Connector:Tag-Connect_TC2030-IDC-NL_2x03_P1.27mm_Vertical -> CircuitPath:ISP_Pads_2x3
